File: keyboard_layout/output/pcbs/combined_board.kicad_pcb (KiCad board)
At the start: 2 copper layers, 309.3 x 113 mm, 132 parts

Commit message: Update final keyboard pcb
Parts:
- removed the ? at (236.8, -36.5)
- removed the ? at (2.00, 11.5)
- removed the ? at (2.00, -68.5)
- removed the ? at (119.3, -60.6)
- removed the ? at (49.4, -36.5)
- removed the ? at (284.2, 11.5)
- removed the ? at (284.2, -68.5)
- removed the ? at (166.9, -60.6)
- added ?: , HOLE_M2_TH, F.Cu at (187.6, -66.7)
- added ?: , HOLE_M2_TH, F.Cu at (208.5, -31.0)
- added ?: , HOLE_M2_TH, F.Cu at (255.8, -37.4)
- added ?: , HOLE_M2_TH, F.Cu at (2.00, 9.53)
- added ?: , HOLE_M2_TH, F.Cu at (7.00, -68.5)
- added ?: , HOLE_M2_TH, F.Cu at (98.6, -66.7)
- added ?: , HOLE_M2_TH, F.Cu at (77.7, -31.0)
- added ?: , HOLE_M2_TH, F.Cu at (30.4, -37.4)
- added ?: , HOLE_M2_TH, F.Cu at (284.2, 9.53)
- added ?: , HOLE_M2_TH, F.Cu at (279.2, -68.5)
- moved MCU2 1.86 mm to (166.8, -48.4)
- moved MCU1 1.86 mm to (119.4, -48.4)
Connections:
- D1 pad 1: P111 -> P115
- D10 pad 1: P113 -> P002
- D11 pad 1: P115 -> P029
- D12 pad 1: P002 -> P031
- D13 pad 1: P111 -> P115
- D14 pad 1: P113 -> P002
- D15 pad 1: P115 -> P029
- D16 pad 1: P002 -> P031
- D17 pad 1: P111 -> P115
- D18 pad 1: P113 -> P002
- D19 pad 1: P115 -> P029
- D2 pad 1: P113 -> P002
- D20 pad 1: P002 -> P031
- D21 pad 1: P111 -> P115
- D22 pad 1: P113 -> P002
- D23 pad 1: P115 -> P029
- D24 pad 1: P002 -> P031
- D25 pad 1: P010 -> P113
- D26 pad 1: P010 -> P113
- D27 pad 1: P010 -> P113
- D28 pad 1: P010 -> P113
- D29 pad 1: P113 -> P002
- D3 pad 1: P115 -> P029
- D30 pad 1: P111 -> P115
- D31 pad 1: P113 -> P002
- D32 pad 1: P115 -> P029
- D33 pad 1: P002 -> P031
- D34 pad 1: P111 -> P115
- D35 pad 1: P113 -> P002
- D36 pad 1: P115 -> P029
- D37 pad 1: P002 -> P031
- D38 pad 1: P111 -> P115
- D39 pad 1: P113 -> P002
- D4 pad 1: P002 -> P031
- D40 pad 1: P115 -> P029
- D41 pad 1: P002 -> P031
- D42 pad 1: P111 -> P115
- D43 pad 1: P113 -> P002
- D44 pad 1: P115 -> P029
- D45 pad 1: P002 -> P031
- D46 pad 1: P111 -> P115
- D47 pad 1: P113 -> P002
- D48 pad 1: P115 -> P029
- D49 pad 1: P002 -> P031
- D5 pad 1: P111 -> P115
- D50 pad 1: P111 -> P115
- D51 pad 1: P113 -> P002
- D52 pad 1: P115 -> P029
- D53 pad 1: P002 -> P031
- D54 pad 1: P010 -> P113
- D55 pad 1: P010 -> P113
- D56 pad 1: P010 -> P113
- D57 pad 1: P010 -> P113
- D58 pad 1: P113 -> P002
- D6 pad 1: P113 -> P002
- D7 pad 1: P115 -> P029
- D8 pad 1: P002 -> P031
- D9 pad 1: P111 -> P115
- S1 pad 1: P006 -> P020
- S10 pad 1: P008 -> P024
- S11 pad 1: P008 -> P024
- S12 pad 1: P008 -> P024
- S13 pad 1: P029 -> P100
- S14 pad 1: P029 -> P100
- S15 pad 1: P029 -> P100
- S16 pad 1: P029 -> P100
- S17 pad 1: P017 -> P011
- S18 pad 1: P017 -> P011
- S19 pad 1: P017 -> P011
- S2 pad 1: P006 -> P020
- S20 pad 1: P017 -> P011
- S21 pad 1: P020 -> P104
- S22 pad 1: P020 -> P104
- S23 pad 1: P020 -> P104
- S24 pad 1: P020 -> P104
- S25 pad 1: P029 -> P100
- S26 pad 1: P017 -> P011
- S27 pad 1: P020 -> P104
- S28 pad 1: P104 -> P017
- S29 pad 1: P104 -> P017
- S3 pad 1: P006 -> P020
- S30 pad 1: P006 -> P020
- S31 pad 1: P006 -> P020
- S32 pad 1: P006 -> P020
- S33 pad 1: P006 -> P020
- S34 pad 1: P031 -> P022
- S35 pad 1: P031 -> P022
- S36 pad 1: P031 -> P022
- S37 pad 1: P031 -> P022
- S38 pad 1: P008 -> P024
- S39 pad 1: P008 -> P024
- S4 pad 1: P006 -> P020
- S40 pad 1: P008 -> P024
- S41 pad 1: P008 -> P024
- S42 pad 1: P029 -> P100
- S43 pad 1: P029 -> P100
- S44 pad 1: P029 -> P100
- S45 pad 1: P029 -> P100
- S46 pad 1: P017 -> P011
- S47 pad 1: P017 -> P011
- S48 pad 1: P017 -> P011
- S49 pad 1: P017 -> P011
- S5 pad 1: P031 -> P022
- S50 pad 1: P020 -> P104
- S51 pad 1: P020 -> P104
- S52 pad 1: P020 -> P104
- S53 pad 1: P020 -> P104
- S54 pad 1: P029 -> P100
- S55 pad 1: P017 -> P011
- S56 pad 1: P020 -> P104
- S57 pad 1: P104 -> P017
- S58 pad 1: P104 -> P017
- S6 pad 1: P031 -> P022
- S7 pad 1: P031 -> P022
- S8 pad 1: P031 -> P022
- S9 pad 1: P008 -> P024
Other:
- board text added: "TINLION"
- board text removed: "TinLion"
